File: Versa64Cart.kicad_pcb (KiCad board)
At the start: 2 copper layers, 57.9 x 48.9 mm, 23 parts, among them J1 EXPANSION_PORT_C64, J2 TEST_1P, J3 TEST_1P, J4 TEST_1P, J5 CONN_02X02, J6 CONN_02X03, SW1 SW_DIP_x05, U1 27512

Commit message: VersaCart logo
Parts:
- added G***: LOGO, Graphics:versacart-logo, F.Cu at (165.1, 76.2)

Commit message: Rev 1.1 - missing trace on ROML
Parts:
- removed the G*** at (165.1, 76.2)
- added G***: LOGO, LOGO, F.Cu at (164.5, 76.2)
Routing:
- net /#ROML: track 50.7 -> 59.9 mm
